Commit message: main

File: install/rm_robot_description/share/rm_robot_description/urdf/simulation_robot.xacro (robot description, xacro)
@@ -1 +1,234 @@
-/home/aurora/RM25/src/rm_robot_description/urdf/simulation_robot.xacro
+<?xml version="1.0"?>
+<robot name="robot" xmlns:xacro="http://www.ros.org/wiki/xacro">
+  <xacro:property name="length_wheel" value="0.05" />
+  <xacro:property name="radius_wheel" value="0.06" />
+  <xacro:property name="PI" value="3.1415926"/>
+  <xacro:macro name="default_inertial" params="mass">
+    <inertial>
+      <mass value="${mass}" />
+      <inertia ixx="0.01" ixy="0.0" ixz="0.0"
+                    iyy="0.01" iyz="0.0" izz="0.01" />
+    </inertial>
+  </xacro:macro>
+  <!-- base_link to livox_frame -->
+  <xacro:arg name="xyz" default="0.12 0.0 0.175" />
+  <xacro:arg name="rpy" default="0 0 0" />
+  <link name="dummy"/>
+  <link name="base_link">
+    <visual>
+      <geometry>
+        <box size="0.2 .3 .1"/>
+      </geometry>
+      <origin rpy="0 0 ${PI/2}" xyz="0 0 0.05"/>
+      <material name="white">
+        <color rgba="1 1 1 1"/>
+      </material>
+    </visual>
+    <collision>
+      <geometry>
+        <box size="0.2 .3 0.1"/>
+      </geometry>
+      <origin rpy="0 0 ${PI/2}" xyz="0 0 0.05"/>
+    </collision>
+    <xacro:default_inertial mass="8.2"/>
+  </link>
+  <joint name="dummy_joint" type="fixed">
+     <parent link="dummy"/>
+     <child link="base_link"/>
+  </joint>
+  <link name="wheel_1">
+    <visual>
+      <geometry>
+        <cylinder length="${length_wheel}" radius="${radius_wheel}"/>
+      </geometry>
+      <origin rpy="0 0 0" xyz="0 0 0"/>
+      <material name="black">
+        <color rgba="0 0 0 1"/>
+      </material>
+    </visual>
+    <collision>
+      <geometry>
+        <cylinder length="${length_wheel}" radius="${radius_wheel}"/>
+      </geometry>
+    </collision>
+    <mu1>0.5</mu1>
+    <mu2>0.5</mu2>
+    <xacro:default_inertial mass="0.5"/>
+  </link>
+  <link name="wheel_2">
+    <visual>
+      <geometry>
+        <cylinder length="${length_wheel}" radius="${radius_wheel}"/>
+      </geometry>
+      <origin rpy="0 0 0" xyz="0 0 0"/>
+      <material name="black"/>
+    </visual>
+    <collision>
+      <geometry>
+        <cylinder length="${length_wheel}" radius="${radius_wheel}"/>
+      </geometry>
+    </collision>
+    <mu1>0.5</mu1>
+    <mu2>0.5</mu2>
+    <xacro:default_inertial mass="0.5"/>
+  </link>
+  <link name="wheel_3">
+    <visual>
+      <geometry>
+        <cylinder length="${length_wheel}" radius="${radius_wheel}"/>
+      </geometry>
+      <origin rpy="0 0 0" xyz="0 0 0"/>
+      <material name="black"/>
+    </visual>
+    <collision>
+      <geometry>
+        <cylinder length="${length_wheel}" radius="${radius_wheel}"/>
+      </geometry>
+    </collision>
+    <mu1>0.5</mu1>
+    <mu2>0.5</mu2>
+    <xacro:default_inertial mass="0.5"/>
+  </link>
+  <link name="wheel_4">
+    <visual>
+      <geometry>
+        <cylinder length="${length_wheel}" radius="${radius_wheel}"/>
+      </geometry>
+      <origin rpy="0 0 0" xyz="0 0 0" />
+      <material name="black"/>
+    </visual>
+    <collision>
+      <geometry>
+        <cylinder length="${length_wheel}" radius="${radius_wheel}"/>
+      </geometry>
+    </collision>
+    <mu1>0.5</mu1>
+    <mu2>0.5</mu2>
+    <xacro:default_inertial mass="0.5"/>
+  </link>
+  <joint name="base_to_wheel1" type="continuous">
+    <parent link="base_link"/>
+    <child link="wheel_1"/>
+    <origin rpy="${-PI/2} 0 0" xyz="0.1 0.13 0"/>
+    <axis xyz="0 0 1" />
+  </joint>
+  <joint name="base_to_wheel2" type="continuous">
+    <axis xyz="0 0 1" />
+    <anchor xyz="0 0 0" />
+    <limit effort="100" velocity="100" />
+    <parent link="base_link"/>
+    <child link="wheel_2"/>
+    <origin rpy="${-PI/2} 0 0" xyz="-0.1 0.13 0"/>
+  </joint>
+  <joint name="base_to_wheel3" type="continuous">
+    <parent link="base_link"/>
+    <axis xyz="0 0 1" />
+    <child link="wheel_3"/>
+    <origin rpy="${-PI/2} 0 0" xyz="0.1 -0.13 0"/>
+  </joint>
+  <joint name="base_to_wheel4" type="continuous">
+    <parent link="base_link"/>
+    <axis xyz="0 0 1" />
+    <child link="wheel_4"/>
+    <origin rpy="${-PI/2} 0 0" xyz="-0.1 -0.13 0"/>
+  </joint>
+  <!-- IMU joint -->
+  <joint name="imu_joint" type="fixed">
+    <axis xyz="0 1 0" />
+    <origin xyz="0.12 0 0.125" rpy="0 0 0"/>
+    <parent link="base_link"/>
+    <child link="imu_link"/>
+  </joint>
+  <!-- IMU -->
+  <link name="imu_link">
+    <collision>
+      <origin xyz="0 0 0" rpy="0 0 0"/>
+      <geometry>
+        <box size="0.05 0.05 0.05"/>
+      </geometry>
+    </collision>
+    <visual>
+      <origin xyz="0 0 0" rpy="0 0 0"/>
+      <geometry>
+        <box size="0.05 0.05 0.05"/>
+      </geometry>
+      <material name="green">
+        <color rgba="0 1 0 1"/>
+      </material>
+    </visual>
+    <inertial>
+      <mass value="1e-2" />
+      <origin xyz="0 0 0" rpy="0 0 0"/>
+      <inertia ixx="1e-6" ixy="0" ixz="0" iyy="1e-6" iyz="0" izz="1e-6" />
+    </inertial>
+  </link>
+  <!-- Gazebo插件设置相关 -->
+  <gazebo reference="base_link">
+    <material>Gazebo/Orange</material>
+  </gazebo>
+  <gazebo reference="wheel_1">
+    <material>Gazebo/Red</material>
+  </gazebo>
+  <gazebo reference="wheel_2">
+    <material>Gazebo/Black</material>
+  </gazebo>
+  <gazebo reference="wheel_3">
+    <material>Gazebo/Red</material>
+  </gazebo>
+  <gazebo reference="wheel_4">
+    <material>Gazebo/Black</material>
+  </gazebo>
+  <gazebo reference="imu_link">
+    <material>Gazebo/BuildingFrame</material>
+  </gazebo>
+  <gazebo reference="livox_frame">
+    <material>Gazebo/LightBlueLaser</material>
+  </gazebo>
+  <!-- Drive controller plugin-->
+  <!-- https://github.com/ros-simulation/gazebo_ros_pkgs/wiki/ROS-2-Migration:-Planar-Move -->
+  <gazebo>
+    <plugin name="mecanum_controller" filename="libgazebo_ros_planar_move.so">
+      <ros>
+        <!-- Add a namespace -->
+        <namespace>/</namespace>
+        <!-- Remap the default topic -->
+        <remapping>cmd_vel:=cmd_vel_chassis</remapping>
+        <remapping>odom:=odom</remapping>
+      </ros>
+      <!-- Set control loop update rate -->
+      <update_rate>100</update_rate>
+      <!-- Set odom publish rate -->
+      <publish_rate>10</publish_rate>
+      <!-- Set if odom required -->
+      <publish_odom>false</publish_odom>
+      <publish_odom_tf>false</publish_odom_tf>
+      <!-- Frame IDs -->
+      <odometry_frame>odom</odometry_frame>
+      <robot_base_frame>base_link</robot_base_frame>
+      <!-- Set odom covariance -->
+      <covariance_x>0.0001</covariance_x>
+      <covariance_y>0.0001</covariance_y>
+      <covariance_yaw>0.01</covariance_yaw>
+    </plugin>
+  </gazebo>
+  <!-- mid360_imu plugin -->
+  <!-- https://github.com/ros-simulation/gazebo_ros_pkgs/wiki/ROS-2-Migration:-IMU-Sensors -->
+  <gazebo reference="imu_link">
+    <sensor name="mid360_imu" type="imu">
+      <always_on>true</always_on>
+      <update_rate>100</update_rate>
+      <plugin name="imu_plugin" filename="libgazebo_ros_imu_sensor.so">
+        <ros>
+          <namespace>/</namespace>
+          <remapping>~/out:=/livox/imu</remapping>
+        </ros>
+        <frame_name>imu_link</frame_name>
+      </plugin>
+    </sensor>
+  </gazebo>
+  <!-- Livox-Mid360  -->
+  <xacro:include filename="$(find ros2_livox_simulation)/urdf/mid360.xacro" />
+  <xacro:mid360 name="livox_frame" parent="base_link" topic="/livox/lidar">
+    <origin xyz="$(arg xyz)" rpy="$(arg rpy)" />
+  </xacro:mid360>
+</robot>
