Commit message: main

File: install/rm_robot_description/share/rm_robot_description/urdf/four_omniwheel_robot.urdf (robot description, URDF)
Before this commit: robot four_omniwheel_robot, 7 links, 6 joints
Links:
- removed link controller_Link
- removed link omniwheel1_Link
- removed link omniwheel2_Link
- removed link omniwheel3_Link
- removed link omniwheel4_Link
- added link controller_link, mass 0; collision mesh filename=package://rm_robot_description/meshes/controller_link.STL; visual mesh filename=package://rm_robot_description/meshes/controller_link.STL
- added link omniwheel1_link, mass 0.43122; collision mesh filename=package://rm_robot_description/meshes/omniwheel1_link.STL; visual mesh filename=package://rm_robot_description/meshes/omniwheel1_link.STL
- added link omniwheel2_link, mass 0.43122; collision mesh filename=package://rm_robot_description/meshes/omniwheel2_link.STL; visual mesh filename=package://rm_robot_description/meshes/omniwheel2_link.STL
- added link omniwheel3_link, mass 0.43122; collision mesh filename=package://rm_robot_description/meshes/omniwheel3_link.STL; visual mesh filename=package://rm_robot_description/meshes/omniwheel3_link.STL
- added link omniwheel4_link, mass 0.431215675623418; collision mesh filename=package://rm_robot_description/meshes/omniwheel4_link.STL; visual mesh filename=package://rm_robot_description/meshes/omniwheel4_link.STL
- link base_link: geometry collision mesh filename=package://rm_robot_description/meshes/base_link.STL; visual mesh filename=package://rm_robot_description/meshes/base_link.STL
- link mid360laser_link: geometry collision mesh filename=package://rm_robot_description/meshes/mid360laser_link.STL; visual mesh filename=package://rm_robot_description/meshes/mid360laser_link.STL
Joints:
- joint controller_joint: child controller_Link -> controller_link
- joint omniwheel1_joint: child omniwheel1_Link -> omniwheel1_link
- joint omniwheel2_joint: child omniwheel2_Link -> omniwheel2_link
- joint omniwheel3_joint: child omniwheel3_Link -> omniwheel3_link
- joint omniwheel4_joint: child omniwheel4_Link -> omniwheel4_link
