Commit message: main

File: src/rm_robot_description/urdf/mid360.xacro (robot description, xacro)
@@ -24,5 +24,5 @@
         <origin xyz="0.025 -0.0265 -0.025" rpy="${pi/2} 0 ${pi}"/>
         <geometry>
-          <mesh filename="model://mid360.stl" scale="0.0008 0.0008 0.0008"/>
+          <mesh filename="file:///home/aurora/RM25/src/rm_robot_description/meshes/mid360.stl" scale="0.0008 0.0008 0.0008"/>
         </geometry>
       </visual>
