Commit message: main

File: src/rm_simulation/rm_robot_description_sim/urdf/mid360.xacro (robot description, xacro)
@@ -4,8 +4,8 @@
   <xacro:property name="laser_min_range" value="0.1"/>
   <xacro:property name="laser_max_range" value="200.0"/>
-  <xacro:property name="samples" value="30000"/>
+  <xacro:property name="samples" value="40000"/>
   <xacro:property name="resolution" value="0.002"/>
   <xacro:property name="noise_mean" value="0.0"/>
-  <xacro:property name="noise_stddev" value="0.002"/>
+  <xacro:property name="noise_stddev" value="0.01"/>
   <xacro:property name="mass" value="0.4" />
   <xacro:property name="length" value="0.1" />
@@ -20,12 +20,12 @@
   </xacro:macro>
   <xacro:macro name="mid360" params="name:='' parent:= 'base_link' topic:='mid360' *origin ">
-    <link name="${name}">
-      <visual>
-        <origin xyz="0.025 -0.0265 0.0" rpy="${pi/2} 0 ${pi}"/>
+<link name="${name}">
+<xacro:box_inertia m="${length}" w="${width}" d="${length}" h="${height}"/>
+  <visual>
         <geometry>
-          <mesh filename="file:///home/aurora/RM25/src/rm_robot_description/meshes/mid360.stl" scale="0.0008 0.0008 0.0008"/>
+            <box size="${length} ${width} ${height}"/>
         </geometry>
-      </visual>
-    </link>
+  </visual>
+</link>
     <joint name="${name}_joint" type="fixed">
       <parent link="${parent}"/>
@@ -38,39 +38,37 @@
         <visualize>true</visualize>
         <update_rate>10</update_rate>
-        <!-- 仿真使用-->
+        <!-- This ray plgin is only for visualization. -->
         <plugin name="${name}_plugin" filename="libros2_livox.so">
-        <!-- 真实使用-->
-        <!-- plugin name="${name}_pluging" filename="libros2_livox.so"-->
-          <ray>
-            <scan>
-              <horizontal>
-                <samples>100</samples>
-                <resolution>1</resolution>
-                <min_angle>${0}</min_angle>
-                <max_angle>${2*M_PI}</max_angle>
-              </horizontal>
-              <vertical>
-                <samples>360</samples>
-                <resolution>1</resolution>
-                <min_angle>${-7.22/180*M_PI}</min_angle>
-                <max_angle>${55.22/180*M_PI}</max_angle>
-              </vertical>
-            </scan>
-            <range>
-              <min>${laser_min_range}</min>
-              <max>${laser_max_range}</max>
-              <resolution>${resolution}</resolution>
-            </range>
-            <noise>
-              <type>gaussian</type>
-              <mean>${noise_mean}</mean>
-              <stddev>${noise_stddev}</stddev>
-            </noise>
-          </ray>
+			<ray>
+			  <scan>
+				<horizontal>
+				<samples>100</samples>
+				<resolution>1</resolution>
+				<min_angle>${0}</min_angle>
+				<max_angle>${2*M_PI}</max_angle>
+				</horizontal>
+				<vertical>
+				<samples>360</samples>
+				<resolution>1</resolution>
+				<min_angle>${-7.22/180*M_PI}</min_angle>
+				<max_angle>${55.22/180*M_PI}</max_angle>
+				</vertical>
+			  </scan>
+			  <range>
+				<min>${laser_min_range}</min>
+				<max>${laser_max_range}</max>
+				<resolution>${resolution}</resolution>
+			  </range>
+			  <noise>
+				<type>gaussian</type>
+				<mean>${noise_mean}</mean>
+				<stddev>${noise_stddev}</stddev>
+			  </noise>
+			</ray>
           <visualize>true</visualize>
-          <samples>${samples}</samples>
-          <downsample>1</downsample>
-          <csv_file_name>$(find rm_robot_description)/scan_mode/mid360.csv</csv_file_name>
-          <topic>${topic}</topic>
+		  <samples>${samples}</samples>
+		  <downsample>1</downsample>
+		  <csv_file_name>$(find ros2_livox_simulation)/scan_mode/mid360.csv</csv_file_name>
+		  <topic>${topic}</topic>
         </plugin>
       </sensor>

File: src/rm_simulation/rm_robot_description_sim/urdf/simulation_waking_robot.xacro (robot description, xacro)
@@ -11,16 +11,8 @@
     </inertial>
   </xacro:macro>
-  <!-- base_link to livox -->
+  <!-- base_link to livox_frame -->
   <xacro:arg name="xyz" default="0.12 0.0 0.175" />
   <xacro:arg name="rpy" default="0 0 0" />
   <link name="dummy"/>
-  <!-- 添加 odom 链接 -->
-  <link name="odom"/>
-  <!-- 从 odom 到 base_link 的固定关节 -->
-  <joint name="odom_to_base" type="fixed">
-    <parent link="odom"/>
-    <child link="base_link"/>
-    <origin xyz="0 0 0" rpy="0 0 0"/>
-  </joint>
   <link name="base_link">
     <visual>
@@ -142,5 +134,5 @@
   </joint>
   <!-- IMU joint -->
-  <joint name="base_to_imu" type="fixed">
+  <joint name="imu_joint" type="fixed">
     <axis xyz="0 1 0" />
     <origin xyz="0.12 0 0.125" rpy="0 0 0"/>
@@ -190,5 +182,5 @@
     <material>Gazebo/BuildingFrame</material>
   </gazebo>
-  <gazebo reference="livox_link">
+  <gazebo reference="livox_frame">
     <material>Gazebo/LightBlueLaser</material>
   </gazebo>
@@ -196,5 +188,5 @@
   <!-- https://github.com/ros-simulation/gazebo_ros_pkgs/wiki/ROS-2-Migration:-Planar-Move -->
   <gazebo>
-    <plugin name="differential_drive_controller" filename="libgazebo_ros_diff_drive.so">
+    <plugin name="mecanum_controller" filename="libgazebo_ros_planar_move.so">
       <ros>
         <!-- Add a namespace -->
@@ -202,5 +194,5 @@
         <!-- Remap the default topic -->
         <remapping>cmd_vel:=cmd_vel_chassis</remapping>
-        <remapping>odom:=/odom</remapping>
+        <remapping>odom:=odom</remapping>
       </ros>
       <!-- Set control loop update rate -->
@@ -237,35 +229,6 @@
   <!-- Livox-Mid360  -->
   <xacro:include filename="$(find ros2_livox_simulation)/urdf/mid360.xacro" />
-  <xacro:mid360 name="livox" parent="base_link" topic="mid360">
+  <xacro:mid360 name="livox_frame" parent="base_link" topic="/livox/lidar">
     <origin xyz="$(arg xyz)" rpy="$(arg rpy)" />
   </xacro:mid360>
-  <!-- Gazebo 插件配置 -->
-<gazebo reference="livox">
-  <plugin name="livox_lidar_plugin" filename="libros2_livox.so">
-    <ros>
-      <namespace>/livox</namespace>
-      <argument>--ros-args</argument>
-    </ros>
-    <topicName>scan</topicName>
-    <frameName>livox</frameName>
-  </plugin>
-</gazebo>
-<gazebo>
-  <plugin name="mecanum_controller" filename="libgazebo_ros_planar_move.so">
-    <ros>
-      <namespace>/</namespace>
-      <remapping>cmd_vel:=/cmd_vel_chassis</remapping>
-      <remapping>odom:=/odom</remapping>
-    </ros>
-    <update_rate>100</update_rate>
-    <publish_rate>10</publish_rate>
-    <publish_odom>false</publish_odom>
-    <publish_odom_tf>false</publish_odom_tf>
-    <odometry_frame>odom</odometry_frame>
-    <robot_base_frame>base_link</robot_base_frame>
-    <covariance_x>0.0001</covariance_x>
-    <covariance_y>0.0001</covariance_y>
-    <covariance_yaw>0.01</covariance_yaw>
-  </plugin>
-</gazebo>
 </robot>

File: src/rm_simulation/ros2_livox_simulation/urdf/mid360.xacro (robot description, xacro)
@@ -14,5 +14,5 @@
   <xacro:macro name="box_inertia" params="m w h d">
     <inertial>
-      <origin xyz="0 0 0" rpy="${pi/2} 0 ${pi/2}"/>
+      <origin xyz="0 0 0" rpy="${M_PI/2} 0 ${M_PI/2}"/>
       <mass value="${m}"/>
       <inertia ixx="${(m/12) * (h*h + d*d)}" ixy="0.0" ixz="0.0" iyy="${(m/12) * (w*w + d*d)}" iyz="0.0" izz="${(m/12) * (w*w + h*h)}"/>
@@ -22,5 +22,5 @@
     <link name="${name}">
       <visual>
-        <origin xyz="0.025 -0.0265 -0.025" rpy="${pi/2} 0 ${pi}"/>
+        <origin xyz="0.025 -0.0265 -0.025" rpy="${M_PI/2} 0 ${M_PI}"/>
         <geometry>
           <mesh filename="model://mid360.stl" scale="0.0008 0.0008 0.0008"/>
